File: kicad/pmod_midi.kicad_pcb (KiCad board)
At the start: 2 copper layers, 24 x 45.6 mm, 14 parts, among them J1 PMOD (12 Pin), J2 Conn_01x02_Pin, Q1 Q_NPN_BCE

Commit message: Added BOM
Parts:
- R4: value 1K -> 1k
- R7: value 10K -> 10k
Other:
- board text added: "ON"
- board text added: "PMOD MIDI 2023 M. J. Dovey"
- board text added: "Rev 1d"
- board text removed: "EN"
- board text removed: "PMOD BLE MIDI 2023 M. J. Dovey"
- board text removed: "Rev 1c"
Changed lines of the file:
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@@
         (effects (font (size 1 1) (thickness 0.15)))
     )
-    (fp_text value "10K" (at 0 1.65) (layer "F.Fab") hide
+    (fp_text value "10k" (at 0 1.65) (layer "F.Fab") hide
         (effects (font (size 1 1) (thickness 0.15)))
     )
@@
         (effects (font (size 1 1) (thickness 0.15)))
     )
-    (fp_text value "1K" (at 0 1.65) (layer "F.Fab") hide
+    (fp_text value "1k" (at 0 1.65) (layer "F.Fab") hide
         (effects (font (size 1 1) (thickness 0.15)))
     )
@@
     (property "Sheetfile" "pmod_midi.kicad_sch")
     (property "Sheetname" "")
+    (property "exclude_from_bom" "")
     (property "ki_description" "Generic connector, single row, 01x02, script generated")
     (property "ki_keywords" "connector")
-    (attr through_hole)
+    (attr through_hole exclude_from_bom)
     (fp_text reference "J2" (at -2.3 0.6) (layer "F.SilkS")
         (effects (font (size 1 1) (thickness 0.15)))
@@
   (gr_rect (start 100 40) (end 124 85.6)
     (stroke (width 0.1) (type default)) (fill none) (layer "Edge.Cuts"))
-  (gr_text "EN" (at 121.87 69.58) (layer "F.SilkS")
+  (gr_text "ON" (at 121.87 69.58) (layer "F.SilkS")
     (effects (font (size 0.8 0.8) (thickness 0.15) bold) (justify bottom))
   )
@@
     (effects (font (size 0.8 0.75) (thickness 0.15) bold) (justify bottom))
   )
-  (gr_text "Rev\n1c\n" (at 121.9 85.3) (layer "F.SilkS")
+  (gr_text "Rev\n1d\n" (at 121.9 85.3) (layer "F.SilkS")
     (effects (font (size 0.8 0.8) (thickness 0.1)) (justify bottom))
   )
@@
     (effects (font (size 0.8 0.8) (thickness 0.15) bold) (justify bottom))
   )
-  (gr_text "PMOD BLE MIDI\n2023 M. J. Dovey" (at 103.3 83 90) (layer "F.SilkS")
+  (gr_text "PMOD MIDI\n2023 M. J. Dovey" (at 103.3 83 90) (layer "F.SilkS")
     (effects (font (size 1 1) (thickness 0.25) bold) (justify left bottom))
   )

Commit message: Updated BOM
Parts:
- removed WIDI1: ~, CME:CME Widi Core Socket
- added J3: CME_Widi_Core_1-8, CME:CME Widi Core Socket Pins 1 - 8, F.Cu at (101.9, 44.3)
- added J4: CME_Widi_Core_9-16, CME:CME Widi Core Socket Pins 9 - 16, F.Cu at (122.1, 44.3)
- added REF**: Standoff Spacer, CME:Standoff Spacer, F.Cu at (122.0, 41.6)
- added REF**: Standoff Spacer, CME:Standoff Spacer, F.Cu at (101.7, 41.7)
- LED1: value LED_ABGR -> LED_ABRG; footprint LED_SMD:LED_Kingbright_AAA3528ESGCT -> LED_SMD:LED_RGB_Wuerth-PLCC4_3.2x2.8mm_150141M173100
Connections:
- LED1 pad 1: /RED -> /V3
- LED1 pad 2: /V3 -> /BLUE
- LED1 pad 3: /BLUE -> /RED
Routing:
- net /GND*: track 55.6 -> 48.3 mm
- net /ON: track 37.0 -> 29.9 mm
- net /RED: track 20.8 -> 20.1 mm
- net /~{BT}: track 34.3 -> 34.9 mm
- net /BT: track 32.0 -> 31.5 mm
- net /BLUE: track 33.4 -> 32.8 mm
- net /GND: vias 2 -> 6
Other:
- board text added: "${PCB-TITLE} ${PCB-YEAR} ${PCB-COMPANY}"
- board text added: "Rev ${PCB-VERSION}${PCB-REVISION}"
- board text added: "VI"
- board text removed: "PMOD MIDI 2023 M. J. Dovey"
- board text removed: "Rev 1d"

Commit message: Updated BOM
Parts:
- removed the REF** at (122.0, 41.6)
- removed the REF** at (101.7, 41.7)
- added H1: MountingHole_Pad, CME:Standoff Spacer, F.Cu at (101.7, 41.7)
- added H2: MountingHole_Pad, CME:Standoff Spacer, F.Cu at (122.0, 41.6)
Changed lines of the file:
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@@
   (net 21 "/RED")
   (net 22 "/BT*")
-  (footprint "CME:Standoff Spacer" (layer "F.Cu")
-    (at 122.025938 41.61975)
-    (attr through_hole board_only)
-    (fp_text reference "REF**" (at 0.43 -2.35 unlocked) (layer "F.SilkS") hide
-        (effects (font (size 1 1) (thickness 0.15)))
-    )
-    (fp_text value "Standoff Spacer" (at 0 1 unlocked) (layer "F.Fab") hide
-        (effects (font (size 1 1) (thickness 0.15)))
-    )
-    (fp_text user "${REFERENCE}" (at 0 2.5 unlocked) (layer "F.Fab") hide
-        (effects (font (size 1 1) (thickness 0.15)))
-    )
-    (fp_circle (center 0.12 0.120354) (end 0.15 -1.149646)
-      (stroke (width 0.05) (type default)) (fill none) (layer "F.CrtYd"))
-    (pad "1" thru_hole circle (at 0.12 0.12) (size 2.5 2.5) (drill 2.2) (layers "*.Cu" "*.Mask")
-      (net 8 "/GND"))
-  )
   (footprint "Resistor_SMD:R_0805_2012Metric_Pad1.20x1.40mm_HandSolder" (layer "F.Cu")
     (at 116.85 57.1)
@@
       (net 7 "/3.3V") (pinfunction "VCC") (pintype "passive"))
   )
-  (footprint "CME:Standoff Spacer" (layer "F.Cu")
-    (at 101.745938 41.65375)
-    (attr through_hole board_only)
-    (fp_text reference "REF**" (at 0.43 -2.35 unlocked) (layer "F.SilkS") hide
-        (effects (font (size 1 1) (thickness 0.15)))
-    )
-    (fp_text value "Standoff Spacer" (at 0 1 unlocked) (layer "F.Fab") hide
-        (effects (font (size 1 1) (thickness 0.15)))
-    )
-    (fp_text user "${REFERENCE}" (at 0 2.5 unlocked) (layer "F.Fab") hide
-        (effects (font (size 1 1) (thickness 0.15)))
-    )
-    (fp_circle (center 0.12 0.120354) (end 0.15 -1.149646)
-      (stroke (width 0.05) (type default)) (fill none) (layer "F.CrtYd"))
-    (pad "1" thru_hole circle (at 0.12 0.12) (size 2.5 2.5) (drill 2.2) (layers "*.Cu" "*.Mask")
-      (net 8 "/GND"))
-  )
   (footprint "Button_Switch_THT:SW_PUSH_6mm" (layer "F.Cu")
     (at 109.9 66.7 -90)
@@
     (property "MPN" "SSW-108-01-L-S")
     (property "Manufacturer" "Samtec")
-    (property "Notes" "1x8 0.1 Inch pitch pin header socket; Optional: 11mm M2 female to female standoff spacer, Two plastic/nylon m2 pan head bolts. For insertion of pins 9-16 of [CME Widi Core module](https://www.cme-pro.com/wp-content/uploads/2022/10/widiCore-Doc-v1.3.pdf).")
+    (property "Notes" "1x8 0.1 Inch pitch pin header socket; . For insertion of pins 9-16 of [CME Widi Core module](https://www.cme-pro.com/wp-content/uploads/2022/10/widiCore-Doc-v1.3.pdf).")
     (property "Sheetfile" "pmod_midi.kicad_sch")
     (property "Sheetname" "")
@@
     (property "MPN" "SSW-108-01-L-S")
     (property "Manufacturer" "Samtec")
-    (property "Notes" "1x8 0.1 Inch pitch pin header socket; Optional: 11mm M2 female to female standoff spacer, Two plastic/nylon m2 pan head bolts. For insertion of pins 1-8 of [CME Widi Core module](https://www.cme-pro.com/wp-content/uploads/2022/10/widiCore-Doc-v1.3.pdf).")
+    (property "Notes" "1x8 0.1 Inch pitch pin header socket; . For insertion of pins 1-8 of [CME Widi Core module](https://www.cme-pro.com/wp-content/uploads/2022/10/widiCore-Doc-v1.3.pdf).")
     (property "Sheetfile" "pmod_midi.kicad_sch")
     (property "Sheetname" "")
@@
     )
   )
+  (footprint "CME:Standoff Spacer" (layer "F.Cu")
+    (at 122.025938 41.619396)
+    (property "MPN" "970100244")
+    (property "Manufacturer" "Würth Elektronik")
+    (property "Notes" "Optional: 10mm M2 female to female standoff spacer, ")
+    (property "Sheetfile" "pmod_midi.kicad_sch")
+    (property "Sheetname" "")
+    (property "ki_description" "Mounting Hole with connection")
+    (property "ki_keywords" "mounting hole")
+    (attr through_hole)
+    (fp_text reference "H2" (at 0.43 -2.35 unlocked) (layer "F.SilkS") hide
+        (effects (font (size 1 1) (thickness 0.15)))
+    )
+    (fp_text value "MountingHole_Pad" (at 0 1 unlocked) (layer "F.Fab") hide
+        (effects (font (size 1 1) (thickness 0.15)))
+    )
+    (fp_text user "${REFERENCE}" (at 0 2.5 unlocked) (layer "F.Fab") hide
+        (effects (font (size 1 1) (thickness 0.15)))
+    )
+    (fp_circle (center 0.12 0.120354) (end 0.15 -1.149646)
+      (stroke (width 0.05) (type default)) (fill none) (layer "F.CrtYd"))
+    (pad "1" thru_hole circle (at 0.12 0.12) (size 2.5 2.5) (drill 2.2) (layers "*.Cu" "*.Mask")
+      (net 8 "/GND") (pinfunction "1") (pintype "input"))
+  )
+  (footprint "CME:Standoff Spacer" (layer "F.Cu")
+    (at 101.745938 41.65375)
+    (property "MPN" "970100244")
+    (property "Manufacturer" "Würth Elektronik")
+    (property "Notes" "Optional: 10mm M2 female to female standoff spacer, ")
+    (property "Sheetfile" "pmod_midi.kicad_sch")
+    (property "Sheetname" "")
+    (property "ki_description" "Mounting Hole with connection")
+    (property "ki_keywords" "mounting hole")
+    (attr through_hole)
+    (fp_text reference "H1" (at 0.43 -2.35 unlocked) (layer "F.SilkS") hide
+        (effects (font (size 1 1) (thickness 0.15)))
+    )
+    (fp_text value "MountingHole_Pad" (at 0 1 unlocked) (layer "F.Fab") hide
+        (effects (font (size 1 1) (thickness 0.15)))
+    )
+    (fp_text user "${REFERENCE}" (at 0 2.5 unlocked) (layer "F.Fab") hide
+        (effects (font (size 1 1) (thickness 0.15)))
+    )
+    (fp_circle (center 0.12 0.120354) (end 0.15 -1.149646)
+      (stroke (width 0.05) (type default)) (fill none) (layer "F.CrtYd"))
+    (pad "1" thru_hole circle (at 0.12 0.12) (size 2.5 2.5) (drill 2.2) (layers "*.Cu" "*.Mask")
+      (net 8 "/GND") (pinfunction "1") (pintype "input"))
+  )
   (footprint "Symbol:OSHW-Logo2_7.3x6mm_SilkScreen" (layer "B.Cu")
