File: kicad/pmod_midi.kicad_sch (KiCad schematic)
At the start: 13 parts, among them J1 PMOD (12 Pin), J2 Conn_01x02_Pin, Q1 Q_NPN_BCE

Commit message: Added BOM
Parts:
- BT1: Part (none) -> 6mm momentarily closed tactile button switch
- J1: Part (none) -> 2x6 0.1 Inch pitch right-angle pin header
- J2: Part (none) -> Optional: 1x2 0.05 Inch pitch pin header
- LED1: value LED_ABGR -> LED_RABG; Part (none) -> 3528 SMD Common Anode RGB LED (Pin order: RABG)
- Q1: Part (none) -> SOT-23 3 SMD NPN Transistor (Pin order: BCE)
- R1, R2, R3, R5, R6: Part (none) -> 0805 SMD Resistor
- R4: value 1K -> 1k; Part (none) -> 0805 SMD Resistor
- R7: value 10K -> 10k; Part (none) -> 0805 SMD Resistor
- WIDI1: value ~ -> CME Widi Core; Part (none) -> Two 1x8 0.1 Inch Pin Header Connector; Optional: Two 11mm M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
Changed lines of the file:
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@@
       (effects (font (size 1.27 1.27)) (justify left) hide)
     )
-    (property "Datasheet" "" (at 140.97 54.61 0)
+    (property "Datasheet" "~" (at 140.97 54.61 0)
       (effects (font (size 1.27 1.27)) (justify left) hide)
+    )
+    (property "Part" "2x6 0.1 Inch pitch right-angle pin header" (at 160.02 54.61 0)
+      (effects (font (size 1.27 1.27)) hide)
     )
     (pin "1")
@@
       (effects (font (size 1.27 1.27)) hide)
     )
+    (property "Part" "SOT-23 3 SMD NPN Transistor (Pin order: BCE)" (at 187.96 90.17 0)
+      (effects (font (size 1.27 1.27)) hide)
+    )
     (pin "1")
     (pin "2")
@@
       (effects (font (size 1.27 1.27)) (justify left))
     )
-    (property "Value" "10K" (at 182.88 95.25 90)
+    (property "Value" "10k" (at 182.88 95.25 90)
       (effects (font (size 1.27 1.27)) (justify left))
     )
@@
     )
     (property "Datasheet" "~" (at 182.88 93.98 0)
+      (effects (font (size 1.27 1.27)) hide)
+    )
+    (property "Part" "0805 SMD Resistor" (at 182.88 93.98 0)
       (effects (font (size 1.27 1.27)) hide)
     )
@@
     )
     (property "Datasheet" "~" (at 203.2 90.17 0)
+      (effects (font (size 1.27 1.27)) hide)
+    )
+    (property "Part" "6mm momentarily closed tactile button switch" (at 198.12 90.17 0)
       (effects (font (size 1.27 1.27)) hide)
     )
@@
       (effects (font (size 1.27 1.27)) (justify right))
     )
-    (property "Value" "LED_ABGR" (at 205.74 38.735 90)
+    (property "Value" "LED_RABG" (at 205.74 38.735 90)
       (effects (font (size 1.27 1.27)) (justify right) hide)
     )
@@
     )
     (property "Datasheet" "~" (at 198.12 36.83 0)
+      (effects (font (size 1.27 1.27)) hide)
+    )
+    (property "Part" "3528 SMD Common Anode RGB LED (Pin order: RABG)" (at 196.85 36.83 90)
       (effects (font (size 1.27 1.27)) hide)
     )
@@
     )
     (property "Datasheet" "~" (at 196.85 44.45 0)
+      (effects (font (size 1.27 1.27)) hide)
+    )
+    (property "Part" "0805 SMD Resistor" (at 196.85 44.45 0)
       (effects (font (size 1.27 1.27)) hide)
     )
@@
       (effects (font (size 1.27 1.27)) (justify left))
     )
-    (property "Value" "~" (at 185.42 63.5 0)
+    (property "Value" "CME Widi Core" (at 185.42 63.5 0)
       (effects (font (size 1.27 1.27)))
     )
@@
     )
     (property "Datasheet" "https://www.cme-pro.com/wp-content/uploads/2022/10/widiCore-Doc-v1.3.pdf" (at 185.42 63.5 0)
+      (effects (font (size 1.27 1.27)) hide)
+    )
+    (property "Part" "Two 1x8 0.1 Inch Pin Header Connector; Optional: Two 11mm M2 Female to Female Standoff Spacers, Four plastic/nylon m2 pan head bolts" (at 190.5 64.77 0)
       (effects (font (size 1.27 1.27)) hide)
     )
@@
       (effects (font (size 1.27 1.27)) hide)
     )
+    (property "Part" "0805 SMD Resistor" (at 194.31 100.33 0)
+      (effects (font (size 1.27 1.27)) hide)
+    )
     (pin "1")
     (pin "2")
@@
       (effects (font (size 1.27 1.27)) hide)
     )
+    (property "Part" "0805 SMD Resistor" (at 182.88 86.36 0)
+      (effects (font (size 1.27 1.27)) hide)
+    )
     (pin "1")
     (pin "2")
@@
       (effects (font (size 1.27 1.27)) hide)
     )
+    (property "Part" "Optional: 1x2 0.05 Inch pitch pin header" (at 168.91 74.93 0)
+      (effects (font (size 1.27 1.27)) hide)
+    )
     (pin "1")
     (pin "2")
@@
       (effects (font (size 1.27 1.27)) hide)
     )
+    (property "Part" "0805 SMD Resistor" (at 191.77 44.45 90)
+      (effects (font (size 1.27 1.27)) hide)
+    )
     (pin "1")
     (pin "2")
@@
       (effects (font (size 1.27 1.27)) (justify left))
     )
-    (property "Value" "1K" (at 154.94 44.45 90)
+    (property "Value" "1k" (at 154.94 44.45 90)
       (effects (font (size 1.27 1.27)) (justify left))
     )
@@
       (effects (font (size 1.27 1.27)) hide)
     )
+    (property "Part" "0805 SMD Resistor" (at 154.94 43.18 90)
+      (effects (font (size 1.27 1.27)) hide)
+    )
     (pin "1")
     (pin "2")
@@
       (effects (font (size 1.27 1.27)) hide)
     )
+    (property "Part" "0805 SMD Resistor" (at 201.93 44.45 0)
+      (effects (font (size 1.27 1.27)) hide)
+    )

Commit message: Tidying
Other:
- title: (none) -> PMOD_MIDI
Changed lines of the file:
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@@
 (kicad_sch (version 20230121) (generator eeschema)
   (paper "A4")
+  (title_block
+    (title "PMOD_MIDI")
+    (date "2023-07-27")
+    (rev "1d")
+  )
   (junction (at 154.94 49.53) (diameter 0) (color 0 0 0 0)
   )

Commit message: Updated BOM
Parts:
- removed LED1: LED_RABG, LED_SMD:LED_Kingbright_AAA3528ESGCT, symbol Device:LED_RABG
- removed WIDI1: CME Widi Core, CME:CME Widi Core Socket, symbol CME:CME_Widi_Core
- added J3: CME_Widi_Core_1-8, CME:CME Widi Core Socket Pins 1 - 8, symbol CME:CME_Widi_Core_1-8
- added J4: CME_Widi_Core_9-16, CME:CME Widi Core Socket Pins 9 - 16, symbol CME:CME_Widi_Core_9-16
- added LED1: LED_ABRG, LED_SMD:LED_RGB_Wuerth-PLCC4_3.2x2.8mm_150141M173100, symbol Device:LED_ABRG
- BT1: MPN (none) -> TS02-66-60-BK-160-LCR-D; Manufacturer (none) -> CUI; Notes (none) -> 6mm momentarily closed tactile button switch; Part 6mm momentarily closed tactile button switch -> (none)
- J1: MPN (none) -> TSW-106-08-L-D-RA; Manufacturer (none) -> Samtec; Notes (none) -> 2x6 0.1 Inch pitch right-angle pin header; Part 2x6 0.1 Inch pitch right-angle pin header -> (none)
- J2: MPN (none) -> 852-10-002-10-001000; Manufacturer (none) -> Mill-Max; Notes (none) -> Optional: 1x2 0.05 Inch pitch pin header; Part Optional: 1x2 0.05 Inch pitch pin header -> (none)
- Q1: MPN (none) -> 2STR2160; Manufacturer (none) -> STMicroelectronics; Notes (none) -> SOT-23 3 SMD NPN Transistor (Pin order: BCE); Part SOT-23 3 SMD NPN Transistor (Pin order: BCE) -> (none)
- R1, R2, R5: MPN (none) -> 680 ohm 0805 SMD Resistor; Part 0805 SMD Resistor -> (none)
- R3: MPN (none) -> 820 ohm 0805 SMD Resistor; Part 0805 SMD Resistor -> (none)
- R4, R6: MPN (none) -> 1k ohm 0805 SMD Resistor; Part 0805 SMD Resistor -> (none)
- R7: MPN (none) -> 10k ohm 0805 SMD Resistor; Part 0805 SMD Resistor -> (none)
Connections:
- net 3.3V: now also J3.7 (VI)
- net BLUE: now also LED1.2 (BK)
- net GND: now also J3.8 (GND)
- net GREEN: now also LED1.4 (GK)
- net LB: now also J3.2 (LB)
- net LG: now also J3.3 (LG)
- net LR: now also J3.4 (LR)
- net ON: now also J3.6 (ON)
- net RED: now also LED1.3 (RK)
- net RX: now also J4.11 (RX)
- net S1: now also J4.16 (S1)
- net S2: now also J4.15 (S2)
- net SF: now also J4.13 (SF)
- net TCK: now also J4.10 (TCK)
- net TMS: now also J4.9 (TMS)
- net TX: now also J3.1 (TX)
- net V3: now also J3.5 (V3), LED1.1 (A)
- net ~{BT}: now also J4.14 (~{BT})
- net ~{RS}: now also J4.12 (~{RS})
Other:
- company: (none) -> ${PCB-COMPANY}
- title: PMOD_MIDI -> ${PCB-TITLE}

Commit message: Updated BOM
Parts:
- added H1, H2: MountingHole_Pad, CME:Standoff Spacer, symbol Mechanical:MountingHole_Pad
- added U1, U2, U3, U4: M2 Nylon Machine Screw, symbol CME:Machine Screw
- J3, J4: Notes 1x8 0.1 Inch pitch pin header socket; Optional: 11mm M2 fem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 -> 1x8 0.1 Inch pitch pin header socket; . For insertion of pi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
Connections:
- net GND: now also H1.1, H2.1
